File: microbit_nrf54l20.kicad_sch (KiCad schematic)
At the start: 66 parts, among them J1 USB_Micro_B, J2 EDGE_CONNECTOR, J3 BAT_2xAAA, SW1 BTN_A, SW2 BTN_B, SW3 RESET, U1 nRF54L20, U2 LSM303C, U3 AP2112K-3.3, Y1 32MHz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

Commit message: Update symbols
Parts:
- removed D1, D10, D11, D12, D13, D14, D15, D16, D17, D18, D19, D2, D20, D21, D22, D23, D24, D25, D3, D4, D5, D6, D7, D8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: LED, LED_SMD:LED_0603_1608Metric, symbol Device:LED
