File: md_nrf54l20-v2.kicad_sch (KiCad schematic)
At the start: 31 parts, among them J1 USB_C, J2 SWD, Q1 BSS138DW, U1 nRF54L20, U2 AMS1117-3.3, U3 CH347T, Y1 8MHz, Y2 32MHz

Commit message: Add CH347 USB schematic with reference-aligned v2
Regenerate the schematic from a kicad-vis circuit description
(circuit.json / circuit_v2.json as the source of truth):
- USB-C -> AMS1117-3.3 -> 3V3; CH347T USB bridge (UART1 to the nRF),
  8 MHz crystal, single-VCC decoupling
- nRF54L20 core: 32 MHz HFXO (12pF C0G loads), DEC/DCC decoupling
- MLT-8530 speaker on a paralleled BSS138DW low-side driver
- 0603 passives (10/22uF bulk stay 0805)
- Hand-authored CH347T symbol added to md_nrf54l20.kicad_sym

v2 (md_nrf54l20-v2.kicad_sch) aligns the nRF power section to the
datasheet reference circuit: DCC inductor 4.7uH, and a 120 ohm ferrite
between DECA and DECRF (each decoupled).

NOTES.md untracked (local build notes only).

Co-Authored-By: Claude Opus 4.8 <noreply@anthropic.com>
Parts:
- added C16: 100nF, Capacitor_SMD:C_0603_1608Metric, symbol Device:C
- added FB1: 120R@100MHz, Inductor_SMD:L_0603_1608Metric, symbol Device:FerriteBead_Small
- L1: value 10uH -> 4.7uH; footprint Inductor_SMD:L_1210_3225Metric -> Inductor_SMD:L_0603_1608Metric
Connections:
- net DECA: now also FB1.1; no longer U1.36 (DECRF)
- net GND: now also C16.2
- new net DECRF: C16.1, FB1.2, U1.36 (DECRF)
Other:
- title: md_nrf54l20 - USB / CH347 / speaker -> md_nrf54l20 - USB / CH347 / speaker (v2, ref-aligned)
- moved on the sheet: L1, R1
