File: md_nrf54l20.kicad_sch (KiCad schematic)
At the start: 37 parts, among them J1 Uno_POWER, J2 Uno_DIGITAL_8_13, J3 Uno_ANALOG, J4 Uno_DIGITAL_0_7, J5 USB_C, J6 SWD, Q1 BSS138DW, U1 nRF54L20, U2 AMS1117-3.3, U3 CH347T, Y1 8MHz, Y2 32MHz

Commit message: Update layout
Parts:
- removed D1: 1N4148, Diode_SMD:D_SOD-123, symbol Device:D
- removed J6: SWD, Connector_PinHeader_2.54mm:PinHeader_1x05_P2.54mm_Vertical, symbol Connector_Generic:Conn_01x05
- removed LS1: MLT-8530, Buzzer_Beeper:MagneticBuzzer_CUI_CMT-8504-100-SMT, symbol Device:Speaker
- removed Q1: BSS138DW, Package_TO_SOT_SMD:SOT-363_SC-70-6, symbol Transistor_FET:Q_Dual_NMOS_S1G1D2S2G2D1
- removed R6: 100k, Resistor_SMD:R_0603_1608Metric, symbol Device:R
- added J6: USB_C, Connector_USB:USB_C_Receptacle_HRO_TYPE-C-31-M-12, symbol Connector:USB_C_Receptacle_USB2.0_16P
- added R4: 5.1k, Resistor_SMD:R_0603_1608Metric, symbol Device:R
- C5: value 1uF -> 2.2uF
- C6: value 1uF -> 4.7uF
- J1: value Uno_POWER -> POWER
- J2: value Uno_DIGITAL_8_13 -> DIGITAL_8_13
- J3: value Uno_ANALOG -> ANALOG
- J4: value Uno_DIGITAL_0_7 -> DIGITAL_0_7
- J5: footprint Connector_USB:USB_C_Receptacle_GCT_USB4105-xx-A_16P_TopMnt_Horizontal -> Connector_USB:USB_C_Receptacle_HRO_TYPE-C-31-M-12
- R5: value 100R -> 5.1k
- U2: footprint Package_TO_SOT_SMD:SOT-223-3_TabPin2 -> Package_TO_SOT_SMD:SOT-89-3
- Y1, Y2: footprint Crystal:Crystal_SMD_3215-2Pin_3.2x1.5mm -> Crystal:Crystal_SMD_3225-4Pin_3.2x2.5mm; symbol Device:Crystal -> Device:Crystal_GND24
Connections:
- net SPK_GATE is gone; now on net GND: R5.2
- net +3V3: no longer L1.2
- net A0: now also U1.7 (P1.29); no longer U1.10 (P1.00)
- net A1: now also U1.8 (P1.30); no longer U1.9 (P1.31)
- net A2: now also U1.9 (P1.31); no longer U1.8 (P1.30)
- net A3: now also U1.10 (P1.00); no longer U1.7 (P1.29)
- net GND: now also Y1.2 (G), Y1.4 (G), Y2.2 (G), Y2.4 (G), J6.A1 (GND), J6.A12 (GND), J6.B1 (GND), J6.B12 (GND), J6.SH (SHIELD), R4.2
- net USB_DP: now also J6.A6 (D+), J6.B6 (D+)
- net VBUS: now also J6.A4 (VBUS), J6.A9 (VBUS), J6.B4 (VBUS), J6.B9 (VBUS)
- net CH_XI: no longer names the net of C12.1, U3.19 (XI), Y1.1
- net CH_XO: no longer names the net of C13.1, U3.20 (XO)
- net CH_XO: now also Y1.3; no longer Y1.2
- net D10_SS renamed D10_CS
- net D11_MOSI renamed D11_COTI
- net D12_MISO renamed D12_CITO
- net DCC: no longer names the net of L1.1, U1.43 (DCC)
- net DECA: no longer names the net of C6.1, FB1.1, U1.46 (DECA)
- net DECD: no longer names the net of C5.1, U1.44 (DECD)
- net DECD: now also L1.2
- net DECRF: no longer names the net of C16.1, FB1.2, U1.36 (DECRF)
- net HFXO_XC1: no longer names the net of C7.1, U1.37 (XC1), Y2.1
- net HFXO_XC2: no longer names the net of C8.1, U1.38 (XC2)
- net HFXO_XC2: now also Y2.3; no longer Y2.2
- net SPK_PWM: no longer names the net of R5.1
- net SPK_PWM: now also J6.A5 (CC1); no longer U1.1 (P2.01)
- net USB_DM renamed USB_DN
- net USB_DN: now also J6.A7 (D-), J6.B7 (D-)
- new net: J6.B5 (CC2), R4.1
- no-connect marks 30 -> 33
Other:
- note added: "VBUS for direct USB communication"
- moved on the sheet: C1, C10, C11, C12, C13, C14, C15, C16, C2, C3, C4, C5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

Commit message: Update layout
Parts:
- added D1: R_LED, LED_SMD:LED_0805_2012Metric, symbol Device:LED
- added D2: O_LED, LED_SMD:LED_0805_2012Metric, symbol Device:LED
- added D3: G_LED, LED_SMD:LED_0805_2012Metric, symbol Device:LED
- added R6: 470, Resistor_SMD:R_0603_1608Metric, symbol Device:R
- added R7: 330, Resistor_SMD:R_0603_1608Metric, symbol Device:R
- added R8: 220, Resistor_SMD:R_0603_1608Metric, symbol Device:R
- added SW1: RESET, md_nrf54l20:micro-switch, symbol Switch:SW_SPST
Connections:
- net +3V3: now also R6.1, R7.1, R8.2
- net GND: now also D1.2 (A), SW1.2 (B)
- net UART_RX: now also D2.2 (A)
- net nRESET: now also SW1.1 (A)
- net at U1.52 (P2.00): now also D3.2 (A)
- new net: D1.1 (K), R6.2
- new net: D3.1 (K), R8.1
- new net: D2.1 (K), R7.2
- no-connect marks 33 -> 32
Other:
- note added: "IS THIS CORRECT?"
- note added: "VBUS for direct USB communication?"
- note removed: "VBUS for direct USB communication"
- moved on the sheet: C1, C10, C11, C12, C13, C14, C15, C16, C2, C3, C4, C5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

Commit message: Update layout
Parts:
- added J7: Conn_01x04, Connectors_JST:JST_SH_SM04B-SRSS-TB_04x1.00mm_Angled, symbol Connector_Generic:Conn_01x04
Connections:
- net +3V3: now also J7.2 (Pin_2)
- net GND: now also J7.1 (Pin_1)
- net at U1.48 (P1.20): now also J7.3 (Pin_3)
- net at U1.49 (P1.21): now also J7.4 (Pin_4)
- no-connect marks 32 -> 30

Commit message: Update layout
Parts:
- added J8: SWD, Connector_PinHeader_2.54mm:PinHeader_1x05_P2.54mm_Vertical, symbol Connector_Generic:Conn_01x05
- added R10, R9: 10k, Resistor_SMD:R_0603_1608Metric, symbol Device:R
Connections:
- net +3V3: now also J8.1 (Pin_1)
- net GND: now also J8.5 (Pin_5), R10.2, R9.2
- net SWDCLK: now also U3.6 (SCK/TCK), J8.3 (Pin_3)
- net SWDIO: now also U3.5 (SCS0/TMS), J8.2 (Pin_2)
- net nRESET: now also U3.9 (SCS1/TRST), J8.4 (Pin_4)
- net MODE_D: now reaches U3.10 (DTR1/MODE0)
- net MODE_D: now also R9.1
- net MODE_R: now reaches U3.13 (RTS1/MODE1)
- net MODE_R: now also R10.1
- no-connect marks 30 -> 28

Commit message: Update layout
Parts:
- removed J1: POWER, Connector_PinSocket_2.54mm:PinSocket_1x08_P2.54mm_Vertical, symbol Connector_Generic:Conn_01x08
- removed J2: DIGITAL_8_13, Connector_PinSocket_2.54mm:PinSocket_1x10_P2.54mm_Vertical, symbol Connector_Generic:Conn_01x10
- removed J3: ANALOG, Connector_PinSocket_2.54mm:PinSocket_1x06_P2.54mm_Vertical, symbol Connector_Generic:Conn_01x06
- removed J4: DIGITAL_0_7, Connector_PinSocket_2.54mm:PinSocket_1x08_P2.54mm_Vertical, symbol Connector_Generic:Conn_01x08
- removed J6: USB_C, Connector_USB:USB_C_Receptacle_HRO_TYPE-C-31-M-12, symbol Connector:USB_C_Receptacle_USB2.0_16P
- removed J8: SWD, Connector_PinHeader_2.54mm:PinHeader_1x05_P2.54mm_Vertical, symbol Connector_Generic:Conn_01x05
- removed R4, R5: 5.1k, Resistor_SMD:R_0603_1608Metric, symbol Device:R
- added J10, J9: Conn_01x15, Connector_PinSocket_2.54mm:PinSocket_1x15_P2.54mm_Vertical, symbol Connector_Generic:Conn_01x15
- added U4: M6017-02, md_nrf54l20:SIM-SMD_M6017-02, symbol md_nrf54l20:M6017-02
- SW1: footprint md_nrf54l20:micro-switch -> md_nrf54l20:QFN-52-1EP_6x6mm_P0.4mm_EP4.7x4.7mm
Connections:
- net +3V3: now also J9.14 (Pin_14)
- net A0: now also J9.12 (Pin_12); no longer U1.7 (P1.29)
- net A1: now also U1.11 (P1.01), J9.11 (Pin_11); no longer U1.8 (P1.30)
- net A2: now also U1.12 (P1.02), J9.10 (Pin_10); no longer U1.9 (P1.31)
- net A3: now also U1.13 (P1.03), J9.9 (Pin_9)
- net A4_SDA: now also J9.8 (Pin_8); no longer U1.16 (P1.06)
- net A5_SCL: now also J9.7 (Pin_7); no longer U1.13 (P1.03)
- net D0_RX: now also J10.2 (Pin_2); no longer U1.23 (P1.08)
- net D10_CS: now also J10.13 (Pin_13); no longer U1.40 (P1.16)
- net D11_COTI: now also J10.14 (Pin_14); no longer U1.41 (P1.18)
- net D12_CITO: now also J10.15 (Pin_15); no longer U1.47 (P1.19)
- net D13_SCK: now also J9.15 (Pin_15); no longer U1.50 (P1.24)
- net D1_TX: now also J10.1 (Pin_1); no longer U1.24 (P1.09)
- net D2: now also J10.5 (Pin_5)
- net D3_PWM: now also J10.6 (Pin_6)
- net D4: now also J10.7 (Pin_7)
- net D5_PWM: now also J10.8 (Pin_8)
- net D6_PWM: now also J10.9 (Pin_9)
- net D7: now also J10.10 (Pin_10); no longer U1.11 (P1.01)
- net D8: now also J10.11 (Pin_11); no longer U1.12 (P1.02)
- net D9_PWM: now also J10.12 (Pin_12); no longer U1.39 (P1.15)
- net GND: now also J10.4 (Pin_4), J9.2 (Pin_2)
- net VBUS: now also J9.4 (Pin_4)
- net nRESET: now also J10.3 (Pin_3), J9.3 (Pin_3)
- net at U1.48 (P1.20): no longer J7.3 (Pin_3)
- net at U1.49 (P1.21): no longer J7.4 (Pin_4)
- net AREF: no longer names the net of U1.22 (P1.07)
- no-connect marks 28 -> 21
Other:
- moved on the sheet: R6, SW1

Commit message: Fix nets in schematic
Parts:
- removed D2: O_LED, LED_SMD:LED_0805_2012Metric, symbol Device:LED
- removed R7: 330, Resistor_SMD:R_0603_1608Metric, symbol Device:R
- J7: value Conn_01x04 -> JST SH I2C
- SW1: footprint md_nrf54l20:QFN-52-1EP_6x6mm_P0.4mm_EP4.7x4.7mm -> Button_Switch_SMD:SW_SPST_EVQP2_MiddlePushTravel_H2.5mm
Connections:
- net +3V3: now also U4.P4 (VDD)
- net A0: now also U1.10 (P1.00)
- net A1: now also U1.9 (P1.31); no longer U1.11 (P1.01)
- net A2: now also U1.8 (P1.30); no longer U1.12 (P1.02)
- net A3: now also U1.7 (P1.29); no longer U1.10 (P1.00), U1.13 (P1.03)
- net A4_SDA: now also U1.16 (P1.06)
- net A5_SCL: now also U1.15 (P1.05)
- net D0_RX: now also U1.47 (P1.19)
- net D10_CS: now also U1.29 (P0.08)
- net D11_COTI: now also U1.28 (P0.07)
- net D12_CITO: now also U1.27 (P0.06)
- net D13_SCK: now also U1.26 (P0.04)
- net D1_TX: now also U1.41 (P1.18)
- net D2: now also U1.40 (P1.16); no longer U1.26 (P0.04)
- net D3_PWM: now also U1.39 (P1.15); no longer U1.27 (P0.06)
- net D4: now also U1.24 (P1.09); no longer U1.28 (P0.07)
- net D5_PWM: now also U1.23 (P1.08); no longer U1.29 (P0.08)
- net D6_PWM: now also U1.22 (P1.07); no longer U1.30 (P0.09)
- net D7: now also U1.14 (P1.04)
- net D8: now also U1.13 (P1.03)
- net D9_PWM: now also U1.30 (P0.09)
- net GND: now also U4.EH, U4.P6 (VSS), U4.SHELL
- net QWIIC_SCL: now also J7.4 (Pin_4), U1.49 (P1.21)
- net QWIIC_SDA: now also J7.3 (Pin_3), U1.48 (P1.20)
- net SD_CS: now also U1.1 (P2.01), U4.P2 (CD/D3)
- net SD_MISO: now also U1.4 (P2.04), U4.P7 (D0)
- net SD_MOSI: now also U1.2 (P2.02), U4.P3 (CMD)
- net SD_SCK: now also U1.5 (P2.05), U4.P5 (CLK)
- net USER_LED: now also D3.2 (A), U1.52 (P2.00)
- net UART_RX: no longer names the net of U3.3 (TXD1)
- net UART_RX: no longer U1.15 (P1.05)
- net UART_TX: no longer names the net of U3.4 (RXD1)
- net UART_TX: no longer U1.14 (P1.04)
- no-connect marks 21 -> 26
Other:
- note removed: "IS THIS CORRECT?"
- moved on the sheet: J10, J7, J9

Commit message: Swap most 0603 to 0402
Parts:
- C11, C12, C13, C14, C15, C16, C2, C3, C4, C5, C7, C8: footprint Capacitor_SMD:C_0603_1608Metric -> Capacitor_SMD:C_0402_1005Metric
- FB1: footprint Inductor_SMD:L_0603_1608Metric -> Inductor_SMD:L_0402_1005Metric
- R1, R10, R2, R3, R6, R8, R9: footprint Resistor_SMD:R_0603_1608Metric -> Resistor_SMD:R_0402_1005Metric
Changed lines of the file:
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@@
 			)
 		)
-		(property "Footprint" "Capacitor_SMD:C_0603_1608Metric"
+		(property "Footprint" "Capacitor_SMD:C_0402_1005Metric"
 			(at 214.63 303.53 0)
 			(hide yes)
@@
 			)
 		)
-		(property "Footprint" "Capacitor_SMD:C_0603_1608Metric"
+		(property "Footprint" "Capacitor_SMD:C_0402_1005Metric"
 			(at 480.06 279.4 0)
 			(hide yes)
@@
 			)
 		)
-		(property "Footprint" "Capacitor_SMD:C_0603_1608Metric"
+		(property "Footprint" "Capacitor_SMD:C_0402_1005Metric"
 			(at 452.12 199.39 0)
 			(hide yes)
@@
 			)
 		)
-		(property "Footprint" "Capacitor_SMD:C_0603_1608Metric"
+		(property "Footprint" "Capacitor_SMD:C_0402_1005Metric"
 			(at 480.06 252.73 0)
 			(hide yes)
@@
 			)
 		)
-		(property "Footprint" "Capacitor_SMD:C_0603_1608Metric"
+		(property "Footprint" "Capacitor_SMD:C_0402_1005Metric"
 			(at 238.76 270.51 0)
 			(hide yes)
@@
 			)
 		)
-		(property "Footprint" "Resistor_SMD:R_0603_1608Metric"
+		(property "Footprint" "Resistor_SMD:R_0402_1005Metric"
 			(at 519.43 228.6 0)
 			(hide yes)
@@
 			)
 		)
-		(property "Footprint" "Resistor_SMD:R_0603_1608Metric"
+		(property "Footprint" "Resistor_SMD:R_0402_1005Metric"
 			(at 227.33 132.08 0)
 			(hide yes)
@@
 			)
 		)
-		(property "Footprint" "Capacitor_SMD:C_0603_1608Metric"
+		(property "Footprint" "Capacitor_SMD:C_0402_1005Metric"
 			(at 214.63 290.83 0)
 			(hide yes)
@@
 			)
 		)
-		(property "Footprint" "Resistor_SMD:R_0603_1608Metric"
+		(property "Footprint" "Resistor_SMD:R_0402_1005Metric"
 			(at 506.73 254 0)
 			(hide yes)
@@
 			)
 		)
-		(property "Footprint" "Resistor_SMD:R_0603_1608Metric"
+		(property "Footprint" "Resistor_SMD:R_0402_1005Metric"
 			(at 299.72 186.69 0)
 			(hide yes)
@@
 			)
 		)
-		(property "Footprint" "Capacitor_SMD:C_0603_1608Metric"
+		(property "Footprint" "Capacitor_SMD:C_0402_1005Metric"
 			(at 251.46 270.51 0)
 			(hide yes)
@@
 			)
 		)
-		(property "Footprint" "Inductor_SMD:L_0603_1608Metric"
+		(property "Footprint" "Inductor_SMD:L_0402_1005Metric"
 			(at 448.31 283.21 0)
 			(hide yes)
@@
 			)
 		)
-		(property "Footprint" "Capacitor_SMD:C_0603_1608Metric"
+		(property "Footprint" "Capacitor_SMD:C_0402_1005Metric"
 			(at 477.52 199.39 0)
 			(hide yes)
@@
 			)
 		)
-		(property "Footprint" "Resistor_SMD:R_0603_1608Metric"
+		(property "Footprint" "Resistor_SMD:R_0402_1005Metric"
 			(at 315 333 0)
 			(hide yes)
@@
 			)
 		)
-		(property "Footprint" "Capacitor_SMD:C_0603_1608Metric"
+		(property "Footprint" "Capacitor_SMD:C_0402_1005Metric"
 			(at 480.06 240.03 0)
 			(hide yes)
@@
 			)
 		)
-		(property "Footprint" "Capacitor_SMD:C_0603_1608Metric"
+		(property "Footprint" "Capacitor_SMD:C_0402_1005Metric"
 			(at 464.82 199.39 0)
 			(hide yes)
@@
 			)
 		)
-		(property "Footprint" "Capacitor_SMD:C_0603_1608Metric"
+		(property "Footprint" "Capacitor_SMD:C_0402_1005Metric"
 			(at 438.15 293.37 0)
 			(hide yes)
@@
 			)
 		)
-		(property "Footprint" "Resistor_SMD:R_0603_1608Metric"
+		(property "Footprint" "Resistor_SMD:R_0402_1005Metric"
 			(at 232.41 132.08 0)
 			(hide yes)
@@
 			)
 		)
-		(property "Footprint" "Capacitor_SMD:C_0603_1608Metric"
+		(property "Footprint" "Capacitor_SMD:C_0402_1005Metric"
 			(at 252.73 194.31 0)
 			(hide yes)
@@
 			)
 		)
-		(property "Footprint" "Resistor_SMD:R_0603_1608Metric"
+		(property "Footprint" "Resistor_SMD:R_0402_1005Metric"
 			(at 330.2 332.74 0)
 			(hide yes)
