File: md_nrf54l20.kicad_sch (KiCad schematic)
At the start: 38 parts, among them J10 Conn_01x15, J5 USB_C, J7 JST SH I2C, J9 Conn_01x15, SW1 RESET, U1 nRF54L20, U2 AMS1117-3.3, U3 CH347T, U4 M6017-02, Y1 8MHz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

Commit message: Remove 10uf filter cap
Parts:
- removed C1: 10uF, Capacitor_SMD:C_0805_2012Metric, symbol Device:C
Changed lines of the file:
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@@
 	)
 	(junction
-		(at 439.42 195.58)
-		(diameter 0)
-		(color 0 0 0 0)
-	)
-	(junction
 		(at 473.71 240.03)
 		(diameter 0)
@@
 	(wire
 		(pts
-			(xy 439.42 195.58) (xy 419.1 195.58)
+			(xy 419.1 195.58) (xy 452.12 195.58)
 		)
 		(stroke
@@
 	(wire
 		(pts
-			(xy 452.12 195.58) (xy 439.42 195.58)
-		)
-		(stroke
-			(width 0)
-			(type default)
-		)
-	)
-	(wire
-		(pts
 			(xy 227.33 190.5) (xy 224.79 190.5)
 		)
@@
 	(symbol
 		(lib_id "power:GND")
-		(at 439.42 203.2 0)
-		(unit 1)
-		(body_style 1)
-		(exclude_from_sim no)
-		(in_bom yes)
-		(on_board yes)
-		(in_pos_files yes)
-		(dnp no)
-		(property "Reference" "#PWR039"
-			(at 439.42 209.55 0)
-			(hide yes)
-			(show_name no)
-			(do_not_autoplace no)
-			(effects
-				(font
-					(size 1.27 1.27)
-				)
-			)
-		)
-		(property "Value" "GND"
-			(at 439.42 207.01 0)
-			(show_name no)
-			(do_not_autoplace no)
-			(effects
-				(font
-					(size 1.27 1.27)
-				)
-			)
-		)
-		(property "Footprint" ""
-			(at 439.42 203.2 0)
-			(hide yes)
-			(show_name no)
-			(do_not_autoplace no)
-			(effects
-				(font
-					(size 1.27 1.27)
-				)
-			)
-		)
-		(property "Datasheet" ""
-			(at 439.42 203.2 0)
-			(hide yes)
-			(show_name no)
-			(do_not_autoplace no)
-			(effects
-				(font
-					(size 1.27 1.27)
-				)
-			)
-		)
-		(property "Description" ""
-			(at 439.42 203.2 0)
-			(hide yes)
-			(show_name no)
-			(do_not_autoplace no)
-			(effects
-				(font
-					(size 1.27 1.27)
-				)
-			)
-		)
-		(pin "1"
-		)
-		(instances
-			(project "md_nrf54l20"
-				(path "/66856a8e-a1ed-409f-881b-bdedd4d4f5ae"
-					(reference "#PWR039")
-					(unit 1)
-				)
-			)
-			(project ""
-				(path "/e09869c8-a609-568e-b6fc-992aa2e6349f"
-					(reference "#PWR039")
-					(unit 1)
-				)
-			)
-		)
-	)
-	(symbol
-		(lib_id "power:GND")
 		(at 480.06 283.21 0)
 		(unit 1)
@@
 					(unit 1)
 				)
-			)
-		)
-	)
-	(symbol
-		(lib_id "Device:C")
-		(at 439.42 199.39 0)
-		(unit 1)
-		(body_style 1)
-		(exclude_from_sim no)
-		(in_bom yes)
-		(on_board yes)
-		(in_pos_files yes)
-		(dnp no)
-		(property "Reference" "C1"
-			(at 434.848 198.39 0)
-			(show_name no)
-			(do_not_autoplace no)
-			(effects
-				(font
-					(size 1.27 1.27)
-				)
-			)
-		)
-		(property "Value" "10uF"
-			(at 433.578 200.39 0)
-			(show_name no)
-			(do_not_autoplace no)
-			(effects
-				(font
-					(size 1.27 1.27)
-				)
-			)
-		)
-		(property "Footprint" "Capacitor_SMD:C_0805_2012Metric"
-			(at 439.42 199.39 0)
-			(hide yes)
-			(show_name no)
-			(do_not_autoplace no)
-			(effects
-				(font
-					(size 1.27 1.27)
-				)
-			)
-		)
-		(property "Datasheet" ""
-			(at 439.42 199.39 0)
-			(hide yes)
-			(show_name no)
-			(do_not_autoplace no)
-			(effects
-				(font
-					(size 1.27 1.27)
-				)
-			)
-		)
-		(property "Description" ""
-			(at 439.42 199.39 0)
-			(hide yes)
-			(show_name no)
-			(do_not_autoplace no)
-			(effects
-				(font
-					(size 1.27 1.27)
-				)
-			)
-		)
-		(pin "1"
-		)
-		(pin "2"
-		)
-		(instances
-			(project "md_nrf54l20"
-				(path "/66856a8e-a1ed-409f-881b-bdedd4d4f5ae"
-					(reference "C1")
-					(unit 1)
-				)
-			)
-			(project ""
-				(path "/e09869c8-a609-568e-b6fc-992aa2e6349f"
-					(reference "C1")
-					(unit 1)
-				)

Commit message: Layout work
Connections:
- net CH_UART_TX: now reaches U3.3 (TXD1)
- net CH_UART_TX: now also U1.50 (P1.24)
- net CH_UART_RX: now reaches U3.4 (RXD1)
- net CH_UART_RX: now also U1.25 (P0.03)
Changed lines of the file:
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@@
-	)
-	(no_connect
-		(at 292.1 283.21)
 	)
 	(no_connect
@@
 	)
 	(no_connect
+		(at 387.35 217.17)
+	)
+	(no_connect
 		(at 201.93 151.13)
 	)
@@
 	)
 	(no_connect
-		(at 292.1 285.75)
-	)
-	(no_connect
 		(at 430.53 269.24)
 	)
@@
 	)
 	(no_connect
+		(at 387.35 219.71)
+	)
+	(no_connect
 		(at 372.11 132.08)
 	)
@@
 	(wire
 		(pts
+			(xy 447.04 214.63) (xy 430.53 214.63)
+		)
+		(stroke
+			(width 0)
+			(type default)
+		)
+	)
+	(wire
+		(pts
 			(xy 265.43 187.96) (xy 265.43 190.5)
 		)
@@
 	(wire
 		(pts
+			(xy 307.34 285.75) (xy 292.1 285.75)
+		)
+		(stroke
+			(width 0)
+			(type default)
+		)
+	)
+	(wire
+		(pts
 			(xy 551.18 318.77) (xy 574.04 318.77)
 		)
@@
 	(wire
 		(pts
+			(xy 374.65 257.81) (xy 394.97 257.81)
+		)
+		(stroke
+			(width 0)
+			(type default)
+		)
+	)
+	(wire
+		(pts
 			(xy 379.73 250.19) (xy 394.97 250.19)
 		)
@@
 		(pts
 			(xy 387.35 217.17) (xy 394.97 217.17)
+		)
+		(stroke
+			(width 0)
+			(type default)
+		)
+	)
+	(wire
+		(pts
+			(xy 307.34 283.21) (xy 292.1 283.21)
 		)
 		(stroke
@@
 		)
 	)
+	(label "CH_UART_TX"
+		(at 374.65 257.81 0)
+		(effects
+			(font
+				(size 1.27 1.27)
+			)
+			(justify left bottom)
+		)
+	)
 	(label "D4"
 		(at 635 323.85 180)
@@
 		)
 	)
+	(label "CH_UART_RX"
+		(at 307.34 285.75 180)
+		(effects
+			(font
+				(size 1.27 1.27)
+			)
+			(justify right bottom)
+		)
+	)
 	(label "MODE_D"
 		(at 314.96 323.85 0)
@@
 		)
 	)
+	(label "CH_UART_TX"
+		(at 307.34 283.21 180)
+		(effects
+			(font
+				(size 1.27 1.27)
+			)
+			(justify right bottom)
+		)
+	)
 	(label "D5_PWM"
 		(at 635 326.39 180)
@@
 		(effects
 			(font
+				(size 1.27 1.27)
+			)
+			(justify right bottom)
+		)
+	)
+	(label "CH_UART_RX"
+		(at 447.04 214.63 180)
+		(effects
+			(font

Commit message: Layout work, all main components on board
Parts:
- C10: value 22uF -> 10uF
Other:
- moved on the sheet: C11

Commit message: More routing, swap jst sh to vertical
Parts:
- J7: footprint Connectors_JST:JST_SH_SM04B-SRSS-TB_04x1.00mm_Angled -> Connector_JST:JST_SH_BM04B-SRSS-TB_1x04-1MP_P1.00mm_Vertical
Changed lines of the file:
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@@
 			)
 		)
-		(property "Footprint" "Connectors_JST:JST_SH_SM04B-SRSS-TB_04x1.00mm_Angled"
+		(property "Footprint" "Connector_JST:JST_SH_BM04B-SRSS-TB_1x04-1MP_P1.00mm_Vertical"
 			(at 328.93 251.46 0)
 			(hide yes)

Commit message: Update layout
Parts:
- added D4: G_LED, LED_SMD:LED_0402_1005Metric, symbol Device:LED
- added D5: O_LED, LED_SMD:LED_0402_1005Metric, symbol Device:LED
- added J1: U.FL Conn, Connector_Coaxial:U.FL_Hirose_U.FL-R-SMT-1_Vertical, symbol Connector:Conn_Coaxial_Small
- added R11, R12: 220, Resistor_SMD:R_0402_1005Metric, symbol Device:R
- D1, D3: footprint LED_SMD:LED_0805_2012Metric -> LED_SMD:LED_0402_1005Metric
- Y1, Y2: footprint Crystal:Crystal_SMD_3225-4Pin_3.2x2.5mm -> Crystal:Crystal_SMD_2016-4Pin_2.0x1.6mm
Connections:
- net +3V3: now also R11.2, R12.2
- net CH_UART_RX: now also D5.1 (K)
- net CH_UART_TX: now also D4.1 (K)
- net GND: now also J1.2 (Ext)
- net at U1.34 (ANT): now also J1.1 (In)
- new net: D4.2 (A), R12.1
- new net: D5.2 (A), R11.1
- no-connect marks 26 -> 25

Commit message: Update layout
Parts:
- SW1: footprint Button_Switch_SMD:SW_SPST_EVQP2_MiddlePushTravel_H2.5mm -> buttons-md:tactile_button_3x2mm
- U4: value M6017-02 -> SD
Connections:
- no-connect marks 25 -> 24
Other:
- note added: "HEADERS"
- note added: "I2C HEADER"
- note added: "SD CARD"
- note added: "USB Controller"
- moved on the sheet: C10, C11, C12, C13, C14, C15, C16, C9, D1, D3, D4, D5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

Commit message: Update layout
Parts:
- U2: value AMS1117-3.3 -> AMS1117 3.3V 1A
Changed lines of the file:
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@@
 			)
 		)
-		(property "Value" "AMS1117-3.3"
+		(property "Value" "AMS1117 3.3V 1A"
 			(at 251.968 152.146 0)
 			(show_name no)

Commit message: Swap mcu direction
Parts:
- removed U2: AMS1117 3.3V 1A, Package_TO_SOT_SMD:SOT-89-3, symbol Regulator_Linear:AMS1117-3.3
- removed U4: SD, md_nrf54l20:SIM-SMD_M6017-02, symbol md_nrf54l20:M6017-02
- added U2: MCP1700x-280xxTT, Package_TO_SOT_SMD:SOT-23, symbol Regulator_Linear:MCP1700x-280xxTT
- added U5: MLD-TF PUSH-H18, md_nrf54l20:TF-SMD_MLD-TF-H15, symbol md_nrf54l20:MLD-TF PUSH-H18
- SW1: footprint buttons-md:tactile_button_3x2mm -> md_nrf54l20:SW-SMD_L3.0-W2.0-LS3.5
Connections:
- net +3V3: now also U2.2 (VO), U5.4 (VDD)
- net GND: now also D1.1 (K), U2.1 (GND), U5.10 (EH), U5.11 (EH), U5.12 (EH), U5.13 (EH), U5.6 (VSS); no longer D1.2 (A)
- net SD_CS: now also U5.2 (CD/DAT3)
- net SD_MISO: now also U5.7 (DAT0)
- net SD_MOSI: now also U5.3 (CMD)
- net SD_SCK: now also U5.5 (CLX)
- net USER_LED: now also D3.1 (K); no longer D3.2 (A)
- net VBUS: now also J9.1 (Pin_1), U2.3 (VI)
- net at R6.2: now also D1.2 (A); no longer D1.1 (K)
- net at R8.1: now also D3.2 (A); no longer D3.1 (K)
- no-connect marks 24 -> 22
Other:
- moved on the sheet: C10, C11, C12, C13, C14, C15, C9, D1, D3, D4, D5, J10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
